File: Hardware/lte_cat_m1_shield_sara-r4.brd (EAGLE design)
At the start: 68.1 x 53.3 mm, 180 parts, among them J8 NANO_SIM, J9 U.FL, Q1 2.5A/30V/105mΩ, Q2 600mA/40V, U1 TXB0104, U2 3.3V, U3 MCP73831, U4 AP7361C-33FGE, U5 SARA-R4

Commit message: Minor revisions post-review
Parts:
- removed U$40: (no value), buzzard_labels:SHIELD38
- added U$102: (no value), buzzard_labels:SOFT#HARD50
- JP2: device SparkFun-Jumpers:SMT-JUMPER_3_NO_NO-SILK -> SparkFun-Jumpers:SMT-JUMPER_3_NO_SILK
- JP3, JP4: value JUMPER-SMT_2_NC_TRACE_NO-SILK -> JUMPER-SMT_2_NC_TRACE_SILK; device SparkFun-Jumpers:SMT-JUMPER_2_NC_TRACE_NO-SILK -> SparkFun-Jumpers:SMT-JUMPER_2_NC_TRACE_SILK
- JP5, JP6: device SparkFun-Jumpers:SMT-JUMPER_2_NC_TRACE_NO-SILK -> SparkFun-Jumpers:SMT-JUMPER_2_NC_TRACE_SILK
- JP7: device SparkFun-Jumpers:SMT-JUMPER_2_NO_NO-SILK -> SparkFun-Jumpers:SMT-JUMPER_2_NO_SILK
- U$11: device buzzard_labels:POWER11 -> buzzard_labels:RESET48
- U$12: device buzzard_labels:RESET10 -> buzzard_labels:GPS47
- U$19: device buzzard_labels:SOFT13 -> buzzard_labels:POWER49
- U$22: device buzzard_labels:HARD12 -> buzzard_labels:SERIAL57
- U$33: device buzzard_labels:GPS30 -> buzzard_labels:ARDUINO51
- U$38: device buzzard_labels:PWR#SEL36 -> buzzard_labels:PWR#SEL53
- U$39: device buzzard_labels:ARDUINO37 -> buzzard_labels:SHIELD52
- U5: value SARA-R4 -> SARA-R410M-2B
- moved U$33 32.0 mm to (9.02, 0.64)
- moved U$19 16.5 mm to (16.3, 47.5)
- moved U$12 15.2 mm to (6.60, 32.5), turned to 90 degrees
- moved U$39 8.40 mm to (17.4, 1.27)
- moved U$11 6.10 mm to (10.3, 47.5)
- moved U$64 5.36 mm to (49.4, 41.8), turned to 90 degrees
- moved U$59 3.53 mm to (39.9, 41.3), turned to 90 degrees
- moved U$22 3.30 mm to (34.7, 48.3)
- moved U$60 3.14 mm to (37.2, 41.7), turned to 90 degrees
- moved U$63 2.62 mm to (42.0, 43.7), turned to 90 degrees
- moved U$76 2.19 mm to (28.5, 4.06), turned to 0 degrees
- moved D5 1.27 mm to (8.26, 19.1)
- moved U$61 1.17 mm to (39.9, 46.4), turned to 90 degrees
- moved U$62 1.17 mm to (37.3, 46.4), turned to 90 degrees
- moved J1 1.14 mm to (5.08, 18.9)
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Routing:
- net SDA-QWIIC: track 30.8 -> 33.2 mm
- net SCL-QWIIC: track 30.3 -> 32.7 mm
- net D_N: track 14.0 -> 12.6 mm
- net GND: track 19.9 -> 21.2 mm
- net D_P: track 15.2 -> 14.0 mm
- net CTS: track 26.8 -> 27.6 mm
- net RTS: track 29.7 -> 30.4 mm
- net 3.3V: track 82.3 -> 83.0 mm
- net VIN: track 30.3 -> 29.7 mm
- net VSIM: track 36.8 -> 37.4 mm
- net SIM_CLK: track 32.4 -> 32.9 mm
Other:
- board text added: "Jim Lindblom"
