File: Hardware/lte_cat_m1_shield_sara-r4.brd (EAGLE design)
At the start: 68.1 x 53.3 mm, 180 parts, among them J8 NANO_SIM, J9 U.FL, Q1 2.5A/30V/105mΩ, Q2 600mA/40V, U1 TXB0104, U2 AP2112K-3.3, U3 MCP73831, U4 AP7361C-33FGE, U5 SARA-R410M-2B

Commit message: v10 of the LTE Shield hardware.
Parts:
- removed U$77: (no value), buzzard_labels:RTS28
- removed U1: TXB0104, SparkFun-IC-Comms:SO14
- added U$40: (no value), buzzard_labels:RST0
- added U6: TCA9406DCU, ublox:VSSOP-8
- added U8: TXB0104, SparkFun-IC-Comms:TSSOP14
- LOGO1: value SPARKX-LOGO4 -> SFE_LOGO_NAME.2_INCH; device SparkX:SPARKX-MEDIUM -> SparkFun-Aesthetics:SFE_LOGO_NAME_.2
- U$42: device buzzard_labels:RTS28 -> buzzard_labels:RST0
- moved LOGO1 8.54 mm to (38.1, 12.7)
- moved C1 4.01 mm to (26.7, 41.3)
- moved C3 4.01 mm to (26.7, 45.1)
- flipped U$42 to the bottom
Connections:
- removed net GPIO3: J4.1, U5.24
- new net GPIO3-CELL: U5.24, U8.2
- new net GPIO3-QWIIC: J4.1, U8.13
- net 1.8V: now also U6.3, U6.6, U8.1, U8.8; no longer U1.1, U1.8
- net D+: now also D5.4, U5.29; no longer D5.6, U5.28
- net D-: now also D5.6, U5.28; no longer D5.4, U5.29
- net GND: now also U6.2, U8.7; no longer U1.7
- net IOREF: now also U6.7, U8.14; no longer U1.14
- net RX-ARDUINO: now also U8.12; no longer U1.11
- net RX-CELL: now also U8.4; no longer U1.5
- net SCL-CELL: now also U6.5; no longer U1.2
- net SCL-QWIIC: now also U6.8; no longer U1.13
- net SDA-CELL: now also U6.4; no longer U1.3
- net SDA-QWIIC: now also U6.1; no longer U1.12
- net TX-ARDUINO: now also U8.11; no longer U1.10
- net TX-CELL: now also U8.3; no longer U1.4
Routing:
- net GPIO3-QWIIC: track 0.00 -> 34.3 mm, vias 0 -> 1
- net GPIO3-CELL: track 0.00 -> 26.3 mm, vias 0 -> 2
- net SDA-QWIIC: track 33.2 -> 27.1 mm
- net GPIO3: track 5.93 -> 0.00 mm
- net IOREF: track 87.7 -> 93.5 mm
- net SCL-QWIIC: track 32.7 -> 28.5 mm
- net 1.8V: track 18.2 -> 20.9 mm, vias 3 -> 2
- net SCL-CELL: track 28.0 -> 29.8 mm
- net SDA-CELL: track 28.0 -> 26.3 mm
- net RX-ARDUINO: track 47.1 -> 45.6 mm, vias 1 -> 2
- net VSIM: track 37.4 -> 36.0 mm
- net D-: track 14.0 -> 12.8 mm
- net D+: track 12.8 -> 14.0 mm
- net TX-CELL: track 10.3 -> 11.3 mm
- net VUSB_DET: track 48.2 -> 49.1 mm
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Other:
- board text added: "v10"
- board text removed: "x01"

Commit message: DNP'ing the antenna-detect circuit.
Parts:
- removed U$32: (no value), buzzard_labels:LTE_CAT_M1#NB_IOT_SHIELD55
- removed U$83: (no value), buzzard_labels:SARA#R410M#02B54
- added U$77: (no value), buzzard_labels:LTE_SHIELD1
- C17: value 27pF -> DNP
- C20: value 33pF -> 0Ohm
- L2: value 68nH -> DNP
- R9: value 10k -> DNP
- moved LOGO1 2.54 mm to (38.1, 10.2)
Changed lines of the file:
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@@
 <attribute name="PROD_ID" value="CAP-00810" x="25.019" y="8.255" size="1.778" layer="27" font="vector" ratio="15" rot="R270" display="off"/>
 </element>
-<element name="C17" library="SparkFun-Capacitors" package="0603" value="27pF" x="45.339" y="30.48">
+<element name="C17" library="SparkFun-Capacitors" package="0603" value="DNP" x="45.339" y="30.48">
 <attribute name="PROD_ID" value="CAP-09989" x="45.339" y="30.48" size="1.778" layer="27" font="vector" ratio="15" display="off"/>
 </element>
-<element name="R9" library="SparkFun-Resistors" package="0603" value="10k" x="44.45" y="32.893" rot="R270">
+<element name="R9" library="SparkFun-Resistors" package="0603" value="DNP" x="44.45" y="32.893" rot="R270">
 <attribute name="PROD_ID" value="RES-00824" x="44.45" y="32.893" size="1.778" layer="27" font="vector" ratio="15" rot="R270" display="off"/>
 </element>
@@
 <attribute name="PROD_ID" value="CAP-07881" x="39.37" y="27.18" size="1.778" layer="27" font="vector" ratio="15" display="off"/>
 </element>
-<element name="C20" library="SparkFun-Capacitors" package="0603" value="33pF" x="44.45" y="27.18">
+<element name="C20" library="SparkFun-Capacitors" package="0603" value="0Ohm" x="44.45" y="27.18">
 <attribute name="PROD_ID" value="CAP-10142" x="44.45" y="27.18" size="1.778" layer="27" font="vector" ratio="15" display="off"/>
 </element>
 <element name="L1" library="ublox" package="0603" value="39nH" x="41.91" y="28.026" rot="R270"/>
-<element name="L2" library="ublox" package="0603" value="68nH" x="46.902" y="28.067" rot="R90"/>
+<element name="L2" library="ublox" package="0603" value="DNP" x="46.902" y="28.067" rot="R90"/>
 <element name="Q2" library="SparkFun-DiscreteSemi" package="SOT23-3" value="600mA/40V" x="3.81" y="29.21" rot="R270">
 <attribute name="PROD_ID" value="TRANS-08049" x="3.81" y="29.21" size="1.778" layer="27" font="vector" ratio="15" rot="R270" display="off"/>
@@
 <element name="FD3" library="SparkFun-Aesthetics" package="FIDUCIAL-MICRO" value="FIDUCIALUFIDUCIAL" x="67.437" y="0.635" rot="MR0"/>
 <element name="FD4" library="SparkFun-Aesthetics" package="FIDUCIAL-MICRO" value="FIDUCIALUFIDUCIAL" x="3.175" y="52.578" rot="MR0"/>
-<element name="U$32" library="buzzard_labels" package="LTE_CAT_M1#NB_IOT_SHIELD55" value="" x="34.29" y="11.43"/>
-<element name="U$83" library="buzzard_labels" package="SARA#R410M#02B54" value="" x="37.846" y="9.525"/>
 <element name="U$102" library="buzzard_labels" package="SOFT#HARD50" value="" x="33.274" y="47.244"/>
 <element name="U$22" library="buzzard_labels" package="SERIAL57" value="" x="34.671" y="48.26"/>
@@
 <element name="U$40" library="buzzard_labels" package="RST0" value="" x="24.13" y="2.921" rot="R90"/>
 <element name="U$42" library="buzzard_labels" package="RST0" value="" x="24.13" y="2.921" rot="MR90"/>
-<element name="LOGO1" library="SparkFun-Aesthetics" package="SFE_LOGO_NAME_.2" value="SFE_LOGO_NAME.2_INCH" x="38.1" y="12.7"/>
+<element name="LOGO1" library="SparkFun-Aesthetics" package="SFE_LOGO_NAME_.2" value="SFE_LOGO_NAME.2_INCH" x="38.1" y="10.16"/>
+<element name="U$77" library="buzzard_labels" package="LTE_SHIELD1" value="" x="41.021" y="10.287"/>
 </elements>
 <signals>
@@
 <contactref element="J1" pad="SHIELD7"/>
 <polygon width="0.254" layer="1" isolate="0.254">
-<vertex x="0" y="14.859"/>
-<vertex x="5.842" y="14.859"/>
-<vertex x="5.842" y="22.733"/>
-<vertex x="0" y="22.733"/>
+<vertex x="0" y="15.113"/>
+<vertex x="5.842" y="15.113"/>
+<vertex x="5.842" y="22.7076"/>
+<vertex x="0" y="22.7076"/>
 </polygon>
 <polygon width="0.254" layer="16" isolate="0.254">
-<vertex x="0" y="14.859"/>
-<vertex x="5.842" y="14.859"/>
-<vertex x="5.842" y="22.733"/>
-<vertex x="0" y="22.733"/>
+<vertex x="0" y="15.113"/>
+<vertex x="5.842" y="15.113"/>
+<vertex x="5.842" y="22.7076"/>
+<vertex x="0" y="22.7076"/>
 </polygon>
 <via x="0.635" y="21.59" extent="1-16" drill="0.3"/>

Commit message: Revisions post-checklist.
Parts:
- removed JP9: J-U.FL, SparkFun-Jumpers:SMT-JUMPER_2_NO_NO-SILK
- removed R9: DNP, SparkFun-Resistors:0603
- added JP1: IOREF-SEL, SparkFun-Jumpers:SMT-JUMPER_3_NO_SILK
- added LOGO3: SFE_LOGO_NAME.2_INCH, SparkFun-Aesthetics:SFE_LOGO_NAME_.2
- added R4: 10k, SparkFun-Resistors:0603
- added U$32: (no value), buzzard_labels:LTE_SHIELD1
- added U$83: (no value), buzzard_labels:HTTPS###SFE#IO#T8160
- C1, C3: value 0.1uF -> 1.0uF
- C16: value 47pF -> DNP
- C17: value DNP -> 47pF
- C19: value 47pF -> 0Ohm
- C2, C4: value 1.0uF -> 0.1uF
- C20: value 0Ohm -> 47pF
- D1: value Yellow -> PRTR5V0U2F; device SparkFun-LED:LED-0603 -> ublox:SOT886
- D2: value 1A/23V/620mV -> Yellow; device SparkFun-DiscreteSemi:SOD-323 -> SparkFun-LED:LED-0603
- D3: value RED -> 1A/23V/620mV; device SparkFun-LED:LED-0603 -> SparkFun-DiscreteSemi:SOD-323
- D4: value BLUE -> RED
- D5: value PRTR5V0U2F -> BLUE; device ublox:SOT886 -> SparkFun-LED:LED-0603
- J8: value NANO_SIM -> U.FL; device ublox:NANO_SIM_WURTH_693043020611 -> SparkFun-Connectors:U.FL
- J9: value U.FL -> NANO_SIM; device SparkFun-Connectors:U.FL -> ublox:NANO_SIM_WURTH_693043020611
- JP2: value IOREF-SEL -> JUMPER-SMT_2_NC_TRACE_SILK; device SparkFun-Jumpers:SMT-JUMPER_3_NO_SILK -> SparkFun-Jumpers:SMT-JUMPER_2_NC_TRACE_SILK
- JP4: value JUMPER-SMT_2_NC_TRACE_SILK -> (none)
- JP6: value (none) -> VUSB_DET; device SparkFun-Jumpers:SMT-JUMPER_2_NC_TRACE_SILK -> SparkFun-Jumpers:SMT-JUMPER_2_NO_SILK
- JP7: value VUSB_DET -> J-CHIP; device SparkFun-Jumpers:SMT-JUMPER_2_NO_SILK -> SparkFun-Jumpers:SMT-JUMPER_2_NC_TRACE_NO-SILK
- JP8: value J-CHIP -> J-U.FL; device SparkFun-Jumpers:SMT-JUMPER_2_NC_TRACE_NO-SILK -> SparkFun-Jumpers:SMT-JUMPER_2_NO_NO-SILK
- R5, R7: value 10k -> 1k
- R6: value 1k -> 10k
- R8: value 1k -> DNP
- U4: value AP7361C-33FGE -> TCA9406DCU; device ublox:8-UDFN -> ublox:VSSOP-8
- U5: value SARA-R410M-2B -> AP7361C-33FGE; device ublox:SARA-LGA -> ublox:8-UDFN
- U6: value TCA9406DCU -> SARA-R410M-2B; device ublox:VSSOP-8 -> ublox:SARA-LGA
- moved FD3 82.6 mm to (3.17, 52.6), flipped to the top
- moved FD4 82.6 mm to (67.4, 0.64), flipped to the top
- moved JP6 43.4 mm to (19.1, 6.35), turned to 270 degrees
- moved JP2 41.1 mm to (39.8, 45.7), turned to 270 degrees
- moved R8 37.6 mm to (44.5, 32.9), turned to 270 degrees
- moved JP7 35.6 mm to (48.5, 26.3), flipped to the top
- moved C16 33.4 mm to (45.3, 30.5), turned to 0 degrees
- moved C17 33.4 mm to (20.4, 8.26), turned to 270 degrees
- moved J8 28.6 mm to (52.7, 27.2), turned to 180 degrees
- moved J9 28.6 mm to (26.7, 15.2), turned to 90 degrees
- moved C19 28.2 mm to (44.5, 27.2), turned to 0 degrees
- moved C20 28.2 mm to (23.5, 8.26), turned to 270 degrees
- moved U4 27.2 mm to (24.1, 43.2)
- moved D2 21.0 mm to (1.91, 25.1)
- moved D3 20.1 mm to (17.5, 11.0), turned to 0 degrees
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- renumbered D7 to D6, U8 to U1
Connections:
- net 1.8V: now also C4.1, U4.3, U4.6, U6.4; no longer C1.1, U5.4, U6.3, U6.6
- net 3.3V: now also C1.1, D5.A, R5.2, U5.1, U6.51, U6.52, U6.53; no longer C2.1, D4.A, R6.2, U4.1, U5.51, U5.52, U5.53
- net ANT: now also U6.56; no longer U5.56
- net ANT_DET: now also R8.1, U6.62; no longer R9.1, U5.62
- net ARDUINO-3.3V: now also JP1.3; no longer JP2.3
- net ARDUINO-5V: now also JP1.1; no longer JP2.1
- net CTS: now also U6.11; no longer U5.11
- net D+: now also D1.4, U6.29; no longer D5.4, U5.29
- net D-: now also D1.6, U6.28; no longer D5.6, U5.28
- net DCD: now also U6.8; no longer U5.8
- net DSR: now also U6.6; no longer U5.6
- net DTR: now also JP5.2, U6.9; no longer JP6.2, U5.9
- net GND: now also C20.2, D1.2, D4.C, J8.1, J8.2, J9.C5, JP4.1, R4.1, U4.2, U5.4, U5.EP, U6.1, U6.14, U6.20, U6.21, U6.22, U6.3, U6.30, U6.32, U6.33, U6.43, U6.5, U6.50, U6.54, U6.55, U6.57, U6.58, U6.59, U6.60, U6.61, U6.63, U6.64, U6.65, U6.66, U6.67, U6.68, U6.69, U6.70, U6.71, U6.72, U6.73, U6.74, U6.75, U6.76, U6.77, U6.78, U6.79, U6.80, U6.81, U6.82, U6.83, U6.84, U6.85, U6.86, U6.87, U6.88, U6.89, U6.90, U6.91, U6.92, U6.93, U6.94, U6.95, U6.96; no longer C19.2, D3.C, D5.2, J8.C5, J9.1, J9.2, JP6.1, R5.1, U4.4, U4.EP, U5.1, U5.14, U5.20, U5.21, U5.22, U5.3, U5.30, U5.32, U5.33, U5.43, U5.5, U5.50, U5.54, U5.55, U5.57, U5.58, U5.59, U5.60, U5.61, U5.63, U5.64, U5.65, U5.66, U5.67, U5.68, U5.69, U5.70, U5.71, U5.72, U5.73, U5.74, U5.75, U5.76, U5.77, U5.78, U5.79, U5.80, U5.81, U5.82, U5.83, U5.84, U5.85, U5.86, U5.87, U5.88, U5.89, U5.90, U5.91, U5.92, U5.93, U5.94, U5.95, U5.96, U6.2
- net GPIO1: now also R6.2, U6.16; no longer R7.2, U5.16
- net GPIO2: now also U6.23; no longer U5.23
- net GPIO3-CELL: now also U6.24; no longer U5.24
- net GPS-3.3V: now also C3.1; no longer C4.1
- net IOREF: now also C2.1, JP1.2, U4.7; no longer C3.1, JP2.2, U6.7
- net N$10: now also R6.1; no longer R7.1
- net N$12: now also D1.1; no longer D5.1
- net N$13: now also D5.C, R7.2; no longer D4.C, R8.2
- net N$14: now also D1.3; no longer D5.3
- net N$15: now also R7.1; no longer R8.1
- net N$16: now also D4.A, R5.1; no longer D3.A, R6.1
- net N$17: now also D2.C; no longer D1.C
- net N$19: now also JP2.1; no longer JP3.1
- net N$20: now also JP3.1; no longer JP4.1
- net N$21: now also C19.2, JP7.1; no longer C20.2, JP9.1
- net N$22: now also JP7.2; no longer JP8.2
- net N$7: now also C16.1, R8.2; no longer C17.1, R9.2
- net N$8: now also C19.1; no longer C20.1
- net N$9: now also J8.FEED, JP8.2; no longer J9.FEED, JP9.2
- net PWR_ON: now also JP2.2, U6.15; no longer JP3.2, U5.15
- net RESET_N: now also JP3.2, U6.18; no longer JP4.2, U5.18
- net RI: now also U6.7; no longer U5.7
- net RTS: now also JP4.2, U6.10; no longer JP5.2, U5.10
- net RX-CELL: now also U6.12; no longer U5.12
- net SCL-CELL: now also U4.5, U6.27; no longer U5.27, U6.5
- net SCL-QWIIC: now also U4.8; no longer U6.8
- net SDA-CELL: now also U4.4, U6.26; no longer U5.26, U6.4
- net SDA-QWIIC: now also U4.1; no longer U6.1
- net SIM_CLK: now also J9.C3, U6.38; no longer J8.C3, U5.38
- net SIM_IO: now also C17.1, J9.C7, U6.39; no longer C16.1, J8.C7, U5.39
- net SIM_RST: now also C20.1, J9.C2, U6.40; no longer C19.1, J8.C2, U5.40
- net TX-CELL: now also U6.13; no longer U5.13
- net VIN: now also D3.C, U5.5, U5.8; no longer D2.C, U4.5, U4.8
- net VSIM: now also J9.C1, U6.41; no longer J8.C1, U5.41
- net VUSB_DET: now also JP6.2, U6.17; no longer JP7.2, U5.17
- net V_USB: now also D1.5, D3.A, JP6.1, R4.2; no longer D1.A, D5.5, JP7.1, R5.2
Routing:
- net 1.8V: track 20.9 -> 21.7 mm
Other:
- board text added: "Units in inches"
