File: Hardware/Production/lte_cat_m1_shield_sara-r4-Panel_v11.brd (EAGLE design)
At the start: 164.3 x 120.9 mm, 718 parts, among them J14 NANO_SIM, J15 U.FL, J23 NANO_SIM, J24 U.FL, J32 NANO_SIM, J33 U.FL, J8 NANO_SIM, J9 U.FL, Q1 2.5A/30V/105mΩ, Q2 600mA/40V, Q3 2.5A/30V/105mΩ, Q4 600mA/40V, Q5 2.5A/30V/105mΩ, Q6 600mA/40V, Q7 2.5A/30V/105mΩ, Q8 600mA/40V, U1 TXB0104, U10 AP2112K-3.3, U11 SARA-R410M-2B, U12 MCP73831, U13 AP7361C-33FGE, U14 TXB0104, U15 AP2112K-3.3, U16 SARA-R410M-2B, U17 MCP73831, U18 AP7361C-33FGE, U19 TXB0104, U2 AP2112K-3.3, U20 AP2112K-3.3, U3 MCP73831, U4 AP7361C-33FGE, U5 SARA-R410M-2B, U6 SARA-R410M-2B, U7 MCP73831, U8 AP7361C-33FGE, U9 TXB0104

Commit message: Production panel v11
Also updated sch pdf
Parts:
- removed E$4: (no value), SparkFun-Aesthetics:FIDUCIAL-1X2
- removed E$5, E$6: (no value), SparkFun-Retired:FIDUCIAL-1.5X3
- added J37: (no value), SparkFun-Connectors:1X06_NO_SILK
- added J38: NANO_SIM, ublox:NANO_SIM_WURTH_693043020611
- added J39: U.FL, SparkFun-Connectors:U.FL
- added J40, J41: (no value), SparkFun-Connectors:1X03_NO_SILK
- added J42: (no value), SparkFun-Connectors:1X01_NO_SILK
- added J43, J44: (no value), SparkFun-Connectors:1X02_NO_SILK
- added LOGO10: OSHW-LOGOM, SparkFun-Aesthetics:OSHW-LOGO-M
- added LOGO11, LOGO12, LOGO9: SFE_LOGO_NAME.2_INCH, SparkFun-Aesthetics:SFE_LOGO_NAME_.2
- added U$413: (no value), buzzard_labels:125
- added U$414: (no value), buzzard_labels:116
- added U$415: (no value), buzzard_labels:107
- added U$416: (no value), buzzard_labels:98
- added U$417: (no value), buzzard_labels:89
- added U$418: (no value), buzzard_labels:714
- added U$419: (no value), buzzard_labels:615
- added U$420: (no value), buzzard_labels:516
- added U$421: (no value), buzzard_labels:417
- added U$422: (no value), buzzard_labels:318
- added U$423: (no value), buzzard_labels:219
- added U$424: (no value), buzzard_labels:TX21
- added U$425: (no value), buzzard_labels:RX22
- added U$426, U$427, U$446: (no value), buzzard_labels:GND3
- added U$428: (no value), buzzard_labels:SOFT#HARD50
- added U$429: (no value), buzzard_labels:SERIAL57
- added U$430: (no value), buzzard_labels:POWER49
- added U$431: (no value), buzzard_labels:RESET48
- added U$432: (no value), buzzard_labels:GPS47
- added U$433: (no value), buzzard_labels:ARDUINO51
- added U$434: (no value), buzzard_labels:SHIELD52
- added U$435: (no value), buzzard_labels:PWR#SEL53
- added U$436, U$437: (no value), buzzard_labels:RST0
- added U$438: (no value), buzzard_labels:HTTPS###SFE#IO#T8160
- added U$439, U$440, U$441, U$442: (no value), buzzard_labels:NC0
- added U$443: (no value), buzzard_labels:GPS#SCL1
- added U$444: (no value), buzzard_labels:GPS#SDA0
- added U$445: (no value), buzzard_labels:VBAT2
- added U$447, U$448: (no value), buzzard_labels:LTE_CAT_M1#NB#IOT_SHIELD1
- added U21: AP7361C-33FGE, ublox:8-UDFN
- added U22: AP2112K-3.3, SparkFun-IC-Power:SOT23-5
- added U23: TCA9406DCU, ublox:VSSOP-8
- added U24: TXB0104, SparkFun-IC-Comms:TSSOP14
- C1, C3: value 0.1uF -> 1.0uF
- C16: value 47pF -> DNP
- C17: value 27pF -> 47pF
- C19: value 47pF -> 0; device SparkFun-Capacitors:0603 -> SparkFun-Resistors:0603
- C2, C4: value 1.0uF -> 0.1uF
- C20: value 33pF -> 47pF
- C31, C51, C71: value 27pF -> DNP
- C33, C53, C73: value 33pF -> 0; device SparkFun-Capacitors:0603 -> SparkFun-Resistors:0603
- D1: value Yellow -> PRTR5V0U2F; device SparkFun-LED:LED-0603 -> ublox:SOT886
- D2: value 1A/23V/620mV -> Yellow; device SparkFun-DiscreteSemi:SOD-323 -> SparkFun-LED:LED-0603
- D3: value RED -> 1A/23V/620mV; device SparkFun-LED:LED-0603 -> SparkFun-DiscreteSemi:SOD-323
- D4: value BLUE -> RED
- D5: value PRTR5V0U2F -> BLUE; device ublox:SOT886 -> SparkFun-LED:LED-0603
- D6: value 1A/23V/620mV -> DT1042-04SO-7; device SparkFun-DiscreteSemi:SOD-323 -> ublox:SOT23-6L
- D7: value DT1042-04SO-7 -> 1A/23V/620mV; device ublox:SOT23-6L -> SparkFun-DiscreteSemi:SOD-323
- E$3: device SparkFun-Aesthetics:FIDUCIAL-1X2 -> SparkFun-Retired:FIDUCIAL-1.5X3
- J10: device SparkFun-Connectors:USB-MICROB-PTH-MILL -> SparkFun-Connectors:1X02_NO_SILK
- J11: device SparkFun-Connectors:1X04_1MM_RA -> SparkFun-Connectors:1X02_NO_SILK
- J12: device SparkFun-Connectors:JST-2-SMD -> SparkFun-Connectors:USB-MICROB-PTH-MILL
- J13: device SparkFun-Connectors:1X06_NO_SILK -> SparkFun-Connectors:1X04_1MM_RA
- J14: value NANO_SIM -> (none); device ublox:NANO_SIM_WURTH_693043020611 -> SparkFun-Connectors:JST-2-SMD
- J15: value U.FL -> (none); device SparkFun-Connectors:U.FL -> SparkFun-Connectors:1X06_NO_SILK
- J16: value (none) -> NANO_SIM; device SparkFun-Connectors:1X03_NO_SILK -> ublox:NANO_SIM_WURTH_693043020611
- J17: value (none) -> U.FL; device SparkFun-Connectors:1X03_NO_SILK -> SparkFun-Connectors:U.FL
- J18: device SparkFun-Connectors:1X01_NO_SILK -> SparkFun-Connectors:1X03_NO_SILK
- J19: device SparkFun-Connectors:USB-MICROB-PTH-MILL -> SparkFun-Connectors:1X03_NO_SILK
- J20: device SparkFun-Connectors:1X04_1MM_RA -> SparkFun-Connectors:1X01_NO_SILK
- J21: device SparkFun-Connectors:JST-2-SMD -> SparkFun-Connectors:1X02_NO_SILK
- J22: device SparkFun-Connectors:1X06_NO_SILK -> SparkFun-Connectors:1X02_NO_SILK
- J23: value NANO_SIM -> (none); device ublox:NANO_SIM_WURTH_693043020611 -> SparkFun-Connectors:USB-MICROB-PTH-MILL
- J24: value U.FL -> (none); device SparkFun-Connectors:U.FL -> SparkFun-Connectors:1X04_1MM_RA
- J25: device SparkFun-Connectors:1X03_NO_SILK -> SparkFun-Connectors:JST-2-SMD
- J26: device SparkFun-Connectors:1X03_NO_SILK -> SparkFun-Connectors:1X06_NO_SILK
- J27: value (none) -> NANO_SIM; device SparkFun-Connectors:1X01_NO_SILK -> ublox:NANO_SIM_WURTH_693043020611
- J28: value (none) -> U.FL; device SparkFun-Connectors:USB-MICROB-PTH-MILL -> SparkFun-Connectors:U.FL
- J29: device SparkFun-Connectors:1X04_1MM_RA -> SparkFun-Connectors:1X03_NO_SILK
- J30: device SparkFun-Connectors:JST-2-SMD -> SparkFun-Connectors:1X03_NO_SILK
- J31: device SparkFun-Connectors:1X06_NO_SILK -> SparkFun-Connectors:1X01_NO_SILK
- J32: value NANO_SIM -> (none); device ublox:NANO_SIM_WURTH_693043020611 -> SparkFun-Connectors:1X02_NO_SILK
- J33: value U.FL -> (none); device SparkFun-Connectors:U.FL -> SparkFun-Connectors:1X02_NO_SILK
- J34: device SparkFun-Connectors:1X03_NO_SILK -> SparkFun-Connectors:USB-MICROB-PTH-MILL
- J35: device SparkFun-Connectors:1X03_NO_SILK -> SparkFun-Connectors:1X04_1MM_RA
- J36: device SparkFun-Connectors:1X01_NO_SILK -> SparkFun-Connectors:JST-2-SMD
- J8: value NANO_SIM -> U.FL; device ublox:NANO_SIM_WURTH_693043020611 -> SparkFun-Connectors:U.FL
- J9: value U.FL -> NANO_SIM; device SparkFun-Connectors:U.FL -> ublox:NANO_SIM_WURTH_693043020611
- JP1: value VUSB_DET -> IOREF-SEL; device SparkFun-Jumpers:SMT-JUMPER_2_NO_SILK -> SparkFun-Jumpers:SMT-JUMPER_3_NO_SILK
- JP2: value IOREF-SEL -> JUMPER-SMT_2_NC_TRACE_SILK; device SparkFun-Jumpers:SMT-JUMPER_3_NO_SILK -> SparkFun-Jumpers:SMT-JUMPER_2_NC_TRACE_SILK
- JP4: value JUMPER-SMT_2_NC_TRACE_SILK -> (none)
- JP6: value (none) -> VUSB_DET; device SparkFun-Jumpers:SMT-JUMPER_2_NC_TRACE_SILK -> SparkFun-Jumpers:SMT-JUMPER_2_NO_SILK
- JP7: value VUSB_DET -> J-CHIP; device SparkFun-Jumpers:SMT-JUMPER_2_NO_SILK -> SparkFun-Jumpers:SMT-JUMPER_2_NC_TRACE_NO-SILK
- JP8: value J-CHIP -> J-U.FL; device SparkFun-Jumpers:SMT-JUMPER_2_NC_TRACE_NO-SILK -> SparkFun-Jumpers:SMT-JUMPER_2_NO_NO-SILK
- JP9: value J-U.FL -> VUSB_DET; device SparkFun-Jumpers:SMT-JUMPER_2_NO_NO-SILK -> SparkFun-Jumpers:SMT-JUMPER_2_NO_SILK
- L2, L4, L6, L8: value 68nH -> DNP
- LOGO1, LOGO3, LOGO5: value SPARKX-LOGO4 -> SFE_LOGO_NAME.2_INCH; device SparkX:SPARKX-MEDIUM -> SparkFun-Aesthetics:SFE_LOGO_NAME_.2
- LOGO6, LOGO8: value OSHW-LOGOM -> SFE_LOGO_NAME.2_INCH; device SparkFun-Aesthetics:OSHW-LOGO-M -> SparkFun-Aesthetics:SFE_LOGO_NAME_.2
- LOGO7: value SPARKX-LOGO4 -> OSHW-LOGOM; device SparkX:SPARKX-MEDIUM -> SparkFun-Aesthetics:OSHW-LOGO-M
- R12, R20, R28: value 10k -> DNP
- R5, R7: value 10k -> 1k
- R6: value 1k -> 10k
- R8: value 1k -> DNP
- U$103: device buzzard_labels:SDA1 -> buzzard_labels:NC0
- U$106: device buzzard_labels:AREF2 -> buzzard_labels:NC0
- U$107: device buzzard_labels:GND3 -> buzzard_labels:NC0
- U$108: device buzzard_labels:134 -> buzzard_labels:NC0
- U$109: device buzzard_labels:125 -> buzzard_labels:GPS#SCL1
- U$110: device buzzard_labels:116 -> buzzard_labels:GPS#SDA0
- U$111: device buzzard_labels:107 -> buzzard_labels:VBAT2
- U$112, U$288: device buzzard_labels:98 -> buzzard_labels:GND3
- U$113: device buzzard_labels:89 -> buzzard_labels:SCL0
- U$114: device buzzard_labels:714 -> buzzard_labels:SDA1
- U$115: device buzzard_labels:615 -> buzzard_labels:AREF2
- U$116: device buzzard_labels:516 -> buzzard_labels:GND3
- U$117: device buzzard_labels:417 -> buzzard_labels:134
- U$118: device buzzard_labels:318 -> buzzard_labels:125
- U$119: device buzzard_labels:219 -> buzzard_labels:116
- U$120, U$232: device buzzard_labels:RX22 -> buzzard_labels:107
- U$121, U$233: device buzzard_labels:TX21 -> buzzard_labels:98
- U$122: device buzzard_labels:CTS23 -> buzzard_labels:89
- U$123: device buzzard_labels:DTR24 -> buzzard_labels:714
- U$124: device buzzard_labels:RI25 -> buzzard_labels:615
- U$125: device buzzard_labels:DSR26 -> buzzard_labels:516
- U$126: device buzzard_labels:DCD27 -> buzzard_labels:417
- U$127, U$239: device buzzard_labels:RTS28 -> buzzard_labels:318
- U$128: device buzzard_labels:VIO29 -> buzzard_labels:219
- U$131: device buzzard_labels:IO334 -> buzzard_labels:CTS23
- U$132: device buzzard_labels:NET31 -> buzzard_labels:DTR24
- U$133: device buzzard_labels:CHG33 -> buzzard_labels:RI25
- U$134: device buzzard_labels:PWR32 -> buzzard_labels:DSR26
- U$135: device buzzard_labels:IOREF39 -> buzzard_labels:DCD27
- U$137: device buzzard_labels:3#3V41 -> buzzard_labels:VIO29
- U$138, U$241: device buzzard_labels:5V42 -> buzzard_labels:RX22
- U$139, U$181, U$242: device buzzard_labels:GND3 -> buzzard_labels:TX21
- U$140: device buzzard_labels:GND3 -> buzzard_labels:IO334
- U$141: device buzzard_labels:VIN43 -> buzzard_labels:NET31
- U$142: device buzzard_labels:A044 -> buzzard_labels:CHG33
- U$143: device buzzard_labels:A145 -> buzzard_labels:PWR32
- U$144: device buzzard_labels:A246 -> buzzard_labels:IOREF39
- U$145: device buzzard_labels:A347 -> buzzard_labels:3#3V41
- U$146: device buzzard_labels:A448 -> buzzard_labels:5V42
- U$147: device buzzard_labels:A549 -> buzzard_labels:GND3
- U$148: device buzzard_labels:NANO50 -> buzzard_labels:GND3
- U$149: device buzzard_labels:SIM51 -> buzzard_labels:VIN43
- U$150: device buzzard_labels:IOREF39 -> buzzard_labels:A044
- U$151, U$375: device buzzard_labels:5V42 -> buzzard_labels:A145
- U$152, U$376: device buzzard_labels:3#3V41 -> buzzard_labels:A246
- U$153: device buzzard_labels:PWR32 -> buzzard_labels:A347
- U$154: device buzzard_labels:RST40 -> buzzard_labels:A448
- U$155: device buzzard_labels:516 -> buzzard_labels:A549
- U$156: device buzzard_labels:615 -> buzzard_labels:NANO50
- U$157: device buzzard_labels:DTR24 -> buzzard_labels:SIM51
- U$158: device buzzard_labels:RTS28 -> buzzard_labels:IOREF39
- U$159: device buzzard_labels:VUSB_DET52 -> buzzard_labels:5V42
- U$160: device buzzard_labels:A549 -> buzzard_labels:3#3V41
- U$161, U$367: device buzzard_labels:A448 -> buzzard_labels:PWR32
- U$162: device buzzard_labels:A347 -> buzzard_labels:RST40
- U$163: device buzzard_labels:A246 -> buzzard_labels:516
- U$164: device buzzard_labels:A145 -> buzzard_labels:615
- U$165: device buzzard_labels:A044 -> buzzard_labels:DTR24
- U$166: device buzzard_labels:VIN43 -> buzzard_labels:RTS28
- U$167: device buzzard_labels:GND3 -> buzzard_labels:VUSB_DET52
- U$168: device buzzard_labels:GND3 -> buzzard_labels:A549
- U$169: device buzzard_labels:5V42 -> buzzard_labels:A448
- U$170: device buzzard_labels:3#3V41 -> buzzard_labels:A347
- U$171: device buzzard_labels:RTS28 -> buzzard_labels:A246
- U$172: device buzzard_labels:IOREF39 -> buzzard_labels:A145
- U$173: device buzzard_labels:IO334 -> buzzard_labels:A044
- U$174: device buzzard_labels:TX21 -> buzzard_labels:VIN43
- U$175, U$400: device buzzard_labels:RX22 -> buzzard_labels:GND3
- U$176, U$334: device buzzard_labels:VIO29 -> buzzard_labels:GND3
- U$177, U$383: device buzzard_labels:SDA1 -> buzzard_labels:5V42
- U$178, U$384: device buzzard_labels:SCL0 -> buzzard_labels:3#3V41
- U$179: device buzzard_labels:AREF2 -> buzzard_labels:IOREF39
- U$180: device buzzard_labels:134 -> buzzard_labels:IO334
- U$182: device buzzard_labels:125 -> buzzard_labels:RX22
- U$183: device buzzard_labels:116 -> buzzard_labels:VIO29
- U$184: device buzzard_labels:107 -> buzzard_labels:SDA1
- U$185: device buzzard_labels:98 -> buzzard_labels:SCL0
- U$186: device buzzard_labels:89 -> buzzard_labels:AREF2
- U$187: device buzzard_labels:714 -> buzzard_labels:134
- U$188, U$259: device buzzard_labels:615 -> buzzard_labels:GND3
- U$189: device buzzard_labels:516 -> buzzard_labels:125
- U$190: device buzzard_labels:417 -> buzzard_labels:116
- U$191: device buzzard_labels:318 -> buzzard_labels:107
- U$192: device buzzard_labels:219 -> buzzard_labels:98
- U$193: device buzzard_labels:TX21 -> buzzard_labels:89
- U$194: device buzzard_labels:RX22 -> buzzard_labels:714
- U$195: device buzzard_labels:GND3 -> buzzard_labels:615
- U$196, U$387: device buzzard_labels:GND3 -> buzzard_labels:516
- U$197: device buzzard_labels:LTE_CAT_M1#NB_IOT_SHIELD55 -> buzzard_labels:417
- U$198: device buzzard_labels:SARA#R410M#02B54 -> buzzard_labels:318
- U$199: device buzzard_labels:SOFT#HARD50 -> buzzard_labels:219
- U$200: device buzzard_labels:SERIAL57 -> buzzard_labels:TX21
- U$201: device buzzard_labels:POWER49 -> buzzard_labels:RX22
- U$202: device buzzard_labels:RESET48 -> buzzard_labels:GND3
- U$203: device buzzard_labels:GPS47 -> buzzard_labels:GND3
- U$204: device buzzard_labels:ARDUINO51 -> buzzard_labels:SOFT#HARD50
- U$205: device buzzard_labels:SHIELD52 -> buzzard_labels:SERIAL57
- U$206: device buzzard_labels:PWR#SEL53 -> buzzard_labels:POWER49
- U$207: device buzzard_labels:SCL0 -> buzzard_labels:RESET48
- U$208: device buzzard_labels:SDA1 -> buzzard_labels:GPS47
- U$209: device buzzard_labels:AREF2 -> buzzard_labels:ARDUINO51
- U$210: device buzzard_labels:GND3 -> buzzard_labels:SHIELD52
- U$211: device buzzard_labels:134 -> buzzard_labels:PWR#SEL53
- U$212: device buzzard_labels:125 -> buzzard_labels:RST0
- U$213: device buzzard_labels:116 -> buzzard_labels:RST0
- U$214: device buzzard_labels:107 -> buzzard_labels:HTTPS###SFE#IO#T8160
- U$215: device buzzard_labels:98 -> buzzard_labels:NC0
- U$216: device buzzard_labels:89 -> buzzard_labels:NC0
- U$217: device buzzard_labels:714 -> buzzard_labels:NC0
- U$218: device buzzard_labels:615 -> buzzard_labels:NC0
- U$219: device buzzard_labels:516 -> buzzard_labels:GPS#SCL1
- U$220: device buzzard_labels:417 -> buzzard_labels:GPS#SDA0
- U$221: device buzzard_labels:318 -> buzzard_labels:VBAT2
- U$222: device buzzard_labels:219 -> buzzard_labels:GND3
- U$223, U$335: device buzzard_labels:RX22 -> buzzard_labels:LTE_CAT_M1#NB#IOT_SHIELD1
- U$224, U$336: device buzzard_labels:TX21 -> buzzard_labels:LTE_CAT_M1#NB#IOT_SHIELD1
- U$225: device buzzard_labels:CTS23 -> buzzard_labels:SCL0
- U$226: device buzzard_labels:DTR24 -> buzzard_labels:SDA1
- U$227: device buzzard_labels:RI25 -> buzzard_labels:AREF2
- U$228: device buzzard_labels:DSR26 -> buzzard_labels:GND3
- U$229: device buzzard_labels:DCD27 -> buzzard_labels:134
- U$230, U$342: device buzzard_labels:RTS28 -> buzzard_labels:125
- U$231: device buzzard_labels:VIO29 -> buzzard_labels:116
- U$234: device buzzard_labels:IO334 -> buzzard_labels:89
- U$235: device buzzard_labels:NET31 -> buzzard_labels:714
- U$236: device buzzard_labels:CHG33 -> buzzard_labels:615
- U$237: device buzzard_labels:PWR32 -> buzzard_labels:516
- U$238: device buzzard_labels:IOREF39 -> buzzard_labels:417
- U$240: device buzzard_labels:3#3V41 -> buzzard_labels:219
- U$243: device buzzard_labels:GND3 -> buzzard_labels:CTS23
- U$244: device buzzard_labels:VIN43 -> buzzard_labels:DTR24
- U$245: device buzzard_labels:A044 -> buzzard_labels:RI25
- U$246: device buzzard_labels:A145 -> buzzard_labels:DSR26
- U$247: device buzzard_labels:A246 -> buzzard_labels:DCD27
- U$248: device buzzard_labels:A347 -> buzzard_labels:RTS28
- U$249: device buzzard_labels:A448 -> buzzard_labels:VIO29
- U$250, U$353: device buzzard_labels:A549 -> buzzard_labels:RX22
- U$251, U$354: device buzzard_labels:NANO50 -> buzzard_labels:TX21
- U$252: device buzzard_labels:SIM51 -> buzzard_labels:IO334
- U$253: device buzzard_labels:IOREF39 -> buzzard_labels:NET31
- U$254: device buzzard_labels:5V42 -> buzzard_labels:CHG33
- U$255, U$273: device buzzard_labels:3#3V41 -> buzzard_labels:PWR32
- U$256: device buzzard_labels:PWR32 -> buzzard_labels:IOREF39
- U$257: device buzzard_labels:RST40 -> buzzard_labels:3#3V41
- U$258: device buzzard_labels:516 -> buzzard_labels:5V42
- U$260: device buzzard_labels:DTR24 -> buzzard_labels:GND3
- U$261: device buzzard_labels:RTS28 -> buzzard_labels:VIN43
- U$262: device buzzard_labels:VUSB_DET52 -> buzzard_labels:A044
- U$263: device buzzard_labels:A549 -> buzzard_labels:A145
- U$264: device buzzard_labels:A448 -> buzzard_labels:A246
- U$266: device buzzard_labels:A246 -> buzzard_labels:A448
- U$267: device buzzard_labels:A145 -> buzzard_labels:A549
- U$268: device buzzard_labels:A044 -> buzzard_labels:NANO50
- U$269: device buzzard_labels:VIN43 -> buzzard_labels:SIM51
- U$270: device buzzard_labels:GND3 -> buzzard_labels:IOREF39
- U$271, U$401: device buzzard_labels:GND3 -> buzzard_labels:5V42
- U$272: device buzzard_labels:5V42 -> buzzard_labels:3#3V41
- U$274: device buzzard_labels:RTS28 -> buzzard_labels:RST40
- U$275: device buzzard_labels:IOREF39 -> buzzard_labels:516
- U$276: device buzzard_labels:IO334 -> buzzard_labels:615
- U$277: device buzzard_labels:TX21 -> buzzard_labels:DTR24
- U$278: device buzzard_labels:RX22 -> buzzard_labels:RTS28
- U$279: device buzzard_labels:VIO29 -> buzzard_labels:VUSB_DET52
- U$280: device buzzard_labels:SDA1 -> buzzard_labels:A549
- U$281: device buzzard_labels:SCL0 -> buzzard_labels:A448
- U$282: device buzzard_labels:AREF2 -> buzzard_labels:A347
- U$283: device buzzard_labels:134 -> buzzard_labels:A246
- U$284: device buzzard_labels:GND3 -> buzzard_labels:A145
- U$285: device buzzard_labels:125 -> buzzard_labels:A044
- U$286: device buzzard_labels:116 -> buzzard_labels:VIN43
- U$287: device buzzard_labels:107 -> buzzard_labels:GND3
- U$289: device buzzard_labels:89 -> buzzard_labels:5V42
- U$290: device buzzard_labels:714 -> buzzard_labels:3#3V41
- U$291: device buzzard_labels:615 -> buzzard_labels:IOREF39
- U$292: device buzzard_labels:516 -> buzzard_labels:IO334
- U$293: device buzzard_labels:417 -> buzzard_labels:TX21
- U$294: device buzzard_labels:318 -> buzzard_labels:RX22
- U$295: device buzzard_labels:219 -> buzzard_labels:VIO29
- U$296: device buzzard_labels:TX21 -> buzzard_labels:SDA1
- U$297: device buzzard_labels:RX22 -> buzzard_labels:SCL0
- U$298: device buzzard_labels:GND3 -> buzzard_labels:AREF2
- U$299: device buzzard_labels:GND3 -> buzzard_labels:134
- U$300: device buzzard_labels:LTE_CAT_M1#NB_IOT_SHIELD55 -> buzzard_labels:GND3
- U$301: device buzzard_labels:SARA#R410M#02B54 -> buzzard_labels:125
- U$302: device buzzard_labels:SOFT#HARD50 -> buzzard_labels:116
- U$303: device buzzard_labels:SERIAL57 -> buzzard_labels:107
- U$304: device buzzard_labels:POWER49 -> buzzard_labels:98
- U$305: device buzzard_labels:RESET48 -> buzzard_labels:89
- U$306: device buzzard_labels:GPS47 -> buzzard_labels:714
- U$307: device buzzard_labels:ARDUINO51 -> buzzard_labels:615
- U$308: device buzzard_labels:SHIELD52 -> buzzard_labels:516
- U$309: device buzzard_labels:PWR#SEL53 -> buzzard_labels:417
- U$310: device buzzard_labels:SCL0 -> buzzard_labels:318
- U$311: device buzzard_labels:SDA1 -> buzzard_labels:219
- U$312: device buzzard_labels:AREF2 -> buzzard_labels:TX21
- U$313: device buzzard_labels:GND3 -> buzzard_labels:RX22
- U$314: device buzzard_labels:134 -> buzzard_labels:GND3
- U$315: device buzzard_labels:125 -> buzzard_labels:GND3
- U$316: device buzzard_labels:116 -> buzzard_labels:SOFT#HARD50
- U$317: device buzzard_labels:107 -> buzzard_labels:SERIAL57
- U$318: device buzzard_labels:98 -> buzzard_labels:POWER49
- U$319: device buzzard_labels:89 -> buzzard_labels:RESET48
- U$32: device buzzard_labels:LTE_CAT_M1#NB_IOT_SHIELD55 -> buzzard_labels:LTE_CAT_M1#NB#IOT_SHIELD1
- U$320: device buzzard_labels:714 -> buzzard_labels:GPS47
- U$321: device buzzard_labels:615 -> buzzard_labels:ARDUINO51
- U$322: device buzzard_labels:516 -> buzzard_labels:SHIELD52
- U$323: device buzzard_labels:417 -> buzzard_labels:PWR#SEL53
- U$324: device buzzard_labels:318 -> buzzard_labels:RST0
- U$325: device buzzard_labels:219 -> buzzard_labels:RST0
- U$326: device buzzard_labels:RX22 -> buzzard_labels:HTTPS###SFE#IO#T8160
- U$327: device buzzard_labels:TX21 -> buzzard_labels:NC0
- U$328: device buzzard_labels:CTS23 -> buzzard_labels:NC0
- U$329: device buzzard_labels:DTR24 -> buzzard_labels:NC0
- U$330: device buzzard_labels:RI25 -> buzzard_labels:NC0
- U$331: device buzzard_labels:DSR26 -> buzzard_labels:GPS#SCL1
- U$332: device buzzard_labels:DCD27 -> buzzard_labels:GPS#SDA0
- U$333: device buzzard_labels:RTS28 -> buzzard_labels:VBAT2
- U$337: device buzzard_labels:IO334 -> buzzard_labels:SCL0
- U$338: device buzzard_labels:NET31 -> buzzard_labels:SDA1
- U$339: device buzzard_labels:CHG33 -> buzzard_labels:AREF2
- U$340: device buzzard_labels:PWR32 -> buzzard_labels:GND3
- U$341: device buzzard_labels:IOREF39 -> buzzard_labels:134
- U$343: device buzzard_labels:3#3V41 -> buzzard_labels:116
- U$344: device buzzard_labels:5V42 -> buzzard_labels:107
- U$345: device buzzard_labels:GND3 -> buzzard_labels:98
- U$346: device buzzard_labels:GND3 -> buzzard_labels:89
- U$347: device buzzard_labels:VIN43 -> buzzard_labels:714
- U$348: device buzzard_labels:A044 -> buzzard_labels:615
- U$349: device buzzard_labels:A145 -> buzzard_labels:516
- U$350: device buzzard_labels:A246 -> buzzard_labels:417
- U$351: device buzzard_labels:A347 -> buzzard_labels:318
- U$352: device buzzard_labels:A448 -> buzzard_labels:219
- U$355: device buzzard_labels:SIM51 -> buzzard_labels:CTS23
- U$356: device buzzard_labels:IOREF39 -> buzzard_labels:DTR24
- U$357: device buzzard_labels:5V42 -> buzzard_labels:RI25
- U$358: device buzzard_labels:3#3V41 -> buzzard_labels:DSR26
- U$359: device buzzard_labels:PWR32 -> buzzard_labels:DCD27
- U$360: device buzzard_labels:RST40 -> buzzard_labels:RTS28
- U$361: device buzzard_labels:516 -> buzzard_labels:VIO29
- U$362: device buzzard_labels:615 -> buzzard_labels:RX22
- U$363: device buzzard_labels:DTR24 -> buzzard_labels:TX21
- U$364: device buzzard_labels:RTS28 -> buzzard_labels:IO334
- U$365: device buzzard_labels:VUSB_DET52 -> buzzard_labels:NET31
- U$366: device buzzard_labels:A549 -> buzzard_labels:CHG33
- U$368: device buzzard_labels:A347 -> buzzard_labels:IOREF39
- U$369: device buzzard_labels:A246 -> buzzard_labels:3#3V41
- U$370: device buzzard_labels:A145 -> buzzard_labels:5V42
- U$371: device buzzard_labels:A044 -> buzzard_labels:GND3
- U$372: device buzzard_labels:VIN43 -> buzzard_labels:GND3
- U$373: device buzzard_labels:GND3 -> buzzard_labels:VIN43
- U$374: device buzzard_labels:GND3 -> buzzard_labels:A044
- U$377: device buzzard_labels:RTS28 -> buzzard_labels:A347
- U$378: device buzzard_labels:IOREF39 -> buzzard_labels:A448
- U$379: device buzzard_labels:IO334 -> buzzard_labels:A549
- U$380: device buzzard_labels:TX21 -> buzzard_labels:NANO50
- U$381: device buzzard_labels:RX22 -> buzzard_labels:SIM51
- U$382: device buzzard_labels:VIO29 -> buzzard_labels:IOREF39
- U$385: device buzzard_labels:AREF2 -> buzzard_labels:PWR32
- U$386: device buzzard_labels:134 -> buzzard_labels:RST40
- U$388: device buzzard_labels:125 -> buzzard_labels:615
- U$389: device buzzard_labels:116 -> buzzard_labels:DTR24
- U$390: device buzzard_labels:107 -> buzzard_labels:RTS28
- U$391: device buzzard_labels:98 -> buzzard_labels:VUSB_DET52
- U$392: device buzzard_labels:89 -> buzzard_labels:A549
- U$393: device buzzard_labels:714 -> buzzard_labels:A448
- U$394: device buzzard_labels:615 -> buzzard_labels:A347
- U$395: device buzzard_labels:516 -> buzzard_labels:A246
- U$396: device buzzard_labels:417 -> buzzard_labels:A145
- U$397: device buzzard_labels:318 -> buzzard_labels:A044
- U$398: device buzzard_labels:219 -> buzzard_labels:VIN43
- U$399: device buzzard_labels:TX21 -> buzzard_labels:GND3
- U$40: device buzzard_labels:SCL0 -> buzzard_labels:RST0
- U$402: device buzzard_labels:GND3 -> buzzard_labels:3#3V41
- U$403: device buzzard_labels:LTE_CAT_M1#NB_IOT_SHIELD55 -> buzzard_labels:IOREF39
- U$404: device buzzard_labels:SARA#R410M#02B54 -> buzzard_labels:IO334
- U$405: device buzzard_labels:SOFT#HARD50 -> buzzard_labels:TX21
- U$406: device buzzard_labels:SERIAL57 -> buzzard_labels:RX22
- U$407: device buzzard_labels:POWER49 -> buzzard_labels:VIO29
- U$408: device buzzard_labels:RESET48 -> buzzard_labels:SDA1
- U$409: device buzzard_labels:GPS47 -> buzzard_labels:SCL0
- U$410: device buzzard_labels:ARDUINO51 -> buzzard_labels:AREF2
- U$411: device buzzard_labels:SHIELD52 -> buzzard_labels:134
- U$412: device buzzard_labels:PWR#SEL53 -> buzzard_labels:GND3
- U$42: device buzzard_labels:RTS28 -> buzzard_labels:RST0
- U$77: device buzzard_labels:RTS28 -> buzzard_labels:LTE_CAT_M1#NB#IOT_SHIELD1
- U$83: device buzzard_labels:SARA#R410M#02B54 -> buzzard_labels:HTTPS###SFE#IO#T8160
- U1: device SparkFun-IC-Comms:SO14 -> SparkFun-IC-Comms:TSSOP14
- U11: value SARA-R410M-2B -> TCA9406DCU; device ublox:SARA-LGA -> ublox:VSSOP-8
- U12: value MCP73831 -> TXB0104; device SparkFun-PowerIC:SOT23-5 -> SparkFun-IC-Comms:TSSOP14
- U13: value AP7361C-33FGE -> SARA-R410M-2B; device ublox:8-UDFN -> ublox:SARA-LGA
- U14: value TXB0104 -> MCP73831; device SparkFun-IC-Comms:SO14 -> SparkFun-PowerIC:SOT23-5
- U15: value AP2112K-3.3 -> AP7361C-33FGE; device SparkFun-IC-Power:SOT23-5 -> ublox:8-UDFN
- U16: value SARA-R410M-2B -> AP2112K-3.3; device ublox:SARA-LGA -> SparkFun-IC-Power:SOT23-5
- U17: value MCP73831 -> TCA9406DCU; device SparkFun-PowerIC:SOT23-5 -> ublox:VSSOP-8
- U18: value AP7361C-33FGE -> TXB0104; device ublox:8-UDFN -> SparkFun-IC-Comms:TSSOP14
- U19: value TXB0104 -> SARA-R410M-2B; device SparkFun-IC-Comms:SO14 -> ublox:SARA-LGA
- U20: value AP2112K-3.3 -> MCP73831; device SparkFun-IC-Power:SOT23-5 -> SparkFun-PowerIC:SOT23-5
- U4: value AP7361C-33FGE -> TCA9406DCU; device ublox:8-UDFN -> ublox:VSSOP-8
- U5: value SARA-R410M-2B -> AP7361C-33FGE; device ublox:SARA-LGA -> ublox:8-UDFN
- U7: value MCP73831 -> SARA-R410M-2B; device SparkFun-PowerIC:SOT23-5 -> ublox:SARA-LGA
- U8: value AP7361C-33FGE -> MCP73831; device ublox:8-UDFN -> SparkFun-PowerIC:SOT23-5
- U9: value TXB0104 -> AP7361C-33FGE; device SparkFun-IC-Comms:SO14 -> ublox:8-UDFN
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Connections:
- removed net GPIO10: R29.2, U16.16
- removed net GPIO11: R32.2, U16.23, U20.3
- removed net GPIO12: J36.1, U16.24
- removed net GPIO9: J27.1, U11.24
- new net GPIO3-CELL: U1.2, U6.24
- new net GPIO3-CELL1: U12.2, U7.24
- new net GPIO3-CELL2: U13.24, U18.2
- new net GPIO3-CELL3: U19.24, U24.2
- new net GPIO3-QWIIC: J4.1, U1.13
- new net GPIO3-QWIIC1: J20.1, U12.13
- new net GPIO3-QWIIC2: J31.1, U18.13
- new net GPIO3-QWIIC3: J42.1, U24.13
- net 1.8V: now also C4.1, U4.3, U4.6, U6.4; no longer C1.1, U5.4
- net 1.8V1: now also U11.3, U11.6, U12.1, U12.8, U7.4; no longer U6.4, U9.1, U9.8
- net 1.8V2: now also U13.4, U17.3, U17.6, U18.1, U18.8; no longer U11.4, U14.1, U14.8
- net 1.8V3: now also U19.4, U23.3, U23.6, U24.1, U24.8; no longer U16.4, U19.1, U19.8
- net 3.3V: now also C1.1, D5.A, R5.2, U5.1, U6.51, U6.52, U6.53; no longer C2.1, D4.A, R6.2, U4.1, U5.51, U5.52, U5.53
- net 3.3V1: now also U7.51, U7.52, U7.53, U9.1; no longer U6.51, U6.52, U6.53, U8.1
- net 3.3V2: now also U13.51, U13.52, U13.53, U16.1; no longer U11.51, U11.52, U11.53, U13.1
- net 3.3V3: now also U19.51, U19.52, U19.53, U21.1, U22.1; no longer U16.51, U16.52, U16.53, U18.1, U20.1
- net ANT: now also U6.56; no longer U5.56
- net ANT1: now also U7.56; no longer U6.56
- net ANT2: now also U13.56; no longer U11.56
- net ANT3: now also U19.56; no longer U16.56
- net ANT_DET: now also R8.1, U6.62; no longer R9.1, U5.62
- net ANT_DET1: now also U7.62; no longer U6.62
- net ANT_DET2: now also U13.62; no longer U11.62
- net ANT_DET3: now also U19.62; no longer U16.62
- net ARDUINO-3.3V: now also JP1.3; no longer JP2.3
- net ARDUINO-5V: now also JP1.1; no longer JP2.1
- net CTS: now also U6.11; no longer U5.11
- net CTS1: now also J19.3, U7.11; no longer J17.3, U6.11
- net CTS2: now also J30.3, U13.11; no longer J26.3, U11.11
- net CTS3: now also J41.3, U19.11; no longer J35.3, U16.11
- net D+: now also D1.4, U6.29; no longer D5.6, U5.28
- net D+1: now also D11.4, U7.29; no longer D11.6, U6.28
- net D+2: now also D17.4, U13.29; no longer D17.6, U11.28
- net D+3: now also D23.4, U19.29; no longer D23.6, U16.28
- net D-: now also D1.6, U6.28; no longer D5.4, U5.29
- net D-1: now also D11.6, U7.28; no longer D11.4, U6.29
- net D-2: now also D17.6, U13.28; no longer D17.4, U11.29
- net D-3: now also D23.6, U19.28; no longer D23.4, U16.29
- net DCD: now also U6.8; no longer U5.8
- net DCD1: now also J18.2, U7.8; no longer J16.2, U6.8
- net DCD2: now also J29.2, U13.8; no longer J25.2, U11.8
- net DCD3: now also J40.2, U19.8; no longer J34.2, U16.8
- net DSR: now also U6.6; no longer U5.6
- net DSR1: now also J18.1, U7.6; no longer J16.1, U6.6
- net DSR2: now also J29.1, U13.6; no longer J25.1, U11.6
- net DSR3: now also J40.1, U19.6; no longer J34.1, U16.6
- net DTR: now also JP5.2, U6.9; no longer JP6.2, U5.9
- net DTR1: now also J19.2, U7.9; no longer J17.2, U6.9
- net DTR2: now also J30.2, U13.9; no longer J26.2, U11.9
- net DTR3: now also J41.2, U19.9; no longer J35.2, U16.9
- net GND: now also C20.2, D1.2, D4.C, D6.2, D6.5, J11.1, J8.1, J8.2, J9.C5, JP4.1, R4.1, U4.2, U5.4, U5.EP, U6.1, U6.14, U6.20, U6.21, U6.22, U6.3, U6.30, U6.32, U6.33, U6.43, U6.5, U6.50, U6.54, U6.55, U6.57, U6.58, U6.59, U6.60, U6.61, U6.63, U6.64, U6.65, U6.66, U6.67, U6.68, U6.69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; no longer B1.AREF, C19.2, D3.C, D5.2, D7.2, D7.5, J8.C5, J9.1, J9.2, JP6.1, R5.1, U4.4, U4.EP, U5.1, U5.14, U5.20, U5.21, U5.22, U5.3, U5.30, U5.32, U5.33, U5.43, U5.5, U5.50, U5.54, U5.55, U5.57, U5.58, U5.59, U5.60, U5.61, U5.63, U5.64, U5.65, U5.66, U5.67, U5.68, U5.69, U5.70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
- net GND1: now also J12.GND, J13.1, J14.1, J15.6, J16.C5, J17.1, J17.2, J22.1, R9.1, U11.2, U12.7, U7.1, U7.14, U7.20, U7.21, U7.22, U7.3, U7.30, U7.32, U7.33, U7.43, U7.5, U7.50, U7.54, U7.55, U7.57, U7.58, U7.59, U7.60, U7.61, U7.63, U7.64, U7.65, U7.66, U7.67, U7.68, U7.69, U7.70, U7.71, U7.72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; no longer B2.AREF, J10.GND, J11.1, J12.1, J13.6, J14.C5, J15.1, J15.2, R4.1, U6.1, U6.14, U6.20, U6.21, U6.22, U6.3, U6.30, U6.32, U6.33, U6.43, U6.5, U6.50, U6.54, U6.55, U6.57, U6.58, U6.59, U6.60, U6.61, U6.63, U6.64, U6.65, U6.66, U6.67, U6.68, U6.69, U6.70, U6.71, U6.72, U6.73, U6.74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
- net GND2: now also J23.GND, J25.1, J26.6, J27.C5, J28.1, J28.2, J33.1, U13.1, U13.14, U13.20, U13.21, U13.22, U13.3, U13.30, U13.32, U13.33, U13.43, U13.5, U13.50, U13.54, U13.55, U13.57, U13.58, U13.59, U13.60, U13.61, U13.63, U13.64, U13.65, U13.66, U13.67, U13.68, U13.69, U13.70, U13.71, U13.72, U13.73, U13.74, U13.75, U13.76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; no longer B3.AREF, J19.GND, J20.1, J21.1, J22.6, J23.C5, J24.2, U11.1, U11.14, U11.20, U11.21, U11.22, U11.3, U11.30, U11.32, U11.33, U11.43, U11.5, U11.50, U11.54, U11.55, U11.57, U11.58, U11.59, U11.60, U11.61, U11.63, U11.64, U11.65, U11.66, U11.67, U11.68, U11.69, U11.70, U11.71, U11.72, U11.73, U11.74, U11.75, U11.76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
- net GND3: now also J34.GND, J35.1, J36.1, J37.6, J38.C5, J39.1, J39.2, J44.1, U19.1, U19.14, U19.20, U19.21, U19.22, U19.3, U19.30, U19.32, U19.33, U19.43, U19.5, U19.50, U19.54, U19.55, U19.57, U19.58, U19.59, U19.60, U19.61, U19.63, U19.64, U19.65, U19.66, U19.67, U19.68, U19.69, U19.70, U19.71, U19.72, U19.73, U19.74, U19.75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; no longer B4.AREF, J28.GND, J29.1, J30.1, J31.6, J32.C5, J33.1, J33.2, U16.1, U16.14, U16.20, U16.21, U16.22, U16.3, U16.30, U16.32, U16.33, U16.43, U16.5, U16.50, U16.54, U16.55, U16.57, U16.58, U16.59, U16.60, U16.61, U16.63, U16.64, U16.65, U16.66, U16.67, U16.68, U16.69, U16.70, U16.71, U16.72, U16.73, U16.74, U16.75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
- net GPIO1: now also R6.2, U6.16; no longer R7.2, U5.16
- net GPIO2: now also U6.23; no longer U5.23
- net GPIO3: now also R13.2, U7.16; no longer J4.1, U5.24
- net GPIO4: now also R16.2, U10.3, U7.23; no longer R13.2, U6.16
- net GPIO5: now also R21.2, U13.16; no longer R16.2, U10.3, U6.23
- net GPIO6: now also R24.2, U13.23, U16.3; no longer J18.1, U6.24
- net GPIO7: now also R29.2, U19.16; no longer R21.2, U11.16
- net GPIO8: now also R32.2, U19.23, U22.3; no longer R24.2, U11.23, U15.3
- net GPS-3.3V: now also C3.1; no longer C4.1
- net GPS-3.3V1: now also J13.2; no longer J11.2
- net GPS-3.3V2: now also J24.2, U16.5; no longer J20.2, U15.5
- net GPS-3.3V3: now also J35.2, U22.5; no longer J29.2, U20.5
- net IOREF: now also C2.1, JP1.2, U4.7; no longer C3.1, JP2.2
- net IOREF1: now also J15.4, U11.7, U12.14; no longer J13.4, U9.14
- net IOREF2: now also J26.4, U17.7, U18.14; no longer J22.4, U14.14
- net IOREF3: now also J37.4, U23.7, U24.14; no longer J31.4, U19.14
- net N$10: now also R6.1; no longer R7.1
- net N$12: now also D1.1; no longer D5.1
- net N$13: now also D5.C, R7.2; no longer D4.C, R8.2
- net N$14: now also D1.3; no longer D5.3
- net N$15: now also R7.1; no longer R8.1
- net N$16: now also D4.A, R5.1; no longer D3.A, R6.1
- net N$17: now also D2.C; no longer D1.C
- net N$19: now also JP2.1; no longer JP3.1
- net N$20: now also JP3.1; no longer JP4.1
- net N$21: now also C19.2, JP7.1; no longer C20.2, JP9.1
- net N$22: now also JP7.2; no longer JP8.2
- net N$23: now also J17.FEED; no longer J15.FEED
- net N$3: now also U8.1; no longer U7.1
- net N$33: now also J12.D-; no longer J10.D-
- net N$34: now also J12.D+; no longer J10.D+
- net N$36: now also U14.1; no longer U12.1
- net N$37: now also U14.5; no longer U12.5
- net N$4: now also U8.5; no longer U7.5
- net N$40: now also J28.FEED; no longer J24.FEED
- net N$50: now also J23.D-; no longer J19.D-
- net N$51: now also J23.D+; no longer J19.D+
- net N$53: now also U20.1; no longer U17.1
- net N$54: now also U20.5; no longer U17.5
- net N$57: now also J39.FEED; no longer J33.FEED
- net N$67: now also J34.D-; no longer J28.D-
- net N$68: now also J34.D+; no longer J28.D+
- net N$7: now also C16.1, R8.2; no longer C17.1, R9.2
- net N$8: now also C19.1; no longer C20.1
- net N$9: now also J8.FEED, JP8.2; no longer J9.FEED, JP9.2
- net PWR_ON: now also JP2.2, U6.15; no longer JP3.2, U5.15
- net PWR_ON1: now also U7.15; no longer U6.15
- net PWR_ON2: now also U13.15; no longer U11.15
- net PWR_ON3: now also U19.15; no longer U16.15
- net RESET_N: now also JP3.2, U6.18; no longer JP4.2, U5.18
- net RESET_N1: now also U7.18; no longer U6.18
- net RESET_N2: now also U13.18; no longer U11.18
- net RESET_N3: now also U19.18; no longer U16.18
- net RI: now also U6.7; no longer U5.7
- net RI1: now also J19.1, U7.7; no longer J17.1, U6.7
- net RI2: now also J30.1, U13.7; no longer J26.1, U11.7
- net RI3: now also J41.1, U19.7; no longer J35.1, U16.7
- net RTS: now also JP4.2, U6.10; no longer JP5.2, U5.10
- net RTS1: now also J18.3, U7.10; no longer J16.3, U6.10
- net RTS2: now also J29.3, U13.10; no longer J25.3, U11.10
- net RTS3: now also J40.3, U19.10; no longer J34.3, U16.10
- net RX-ARDUINO: now also U1.12; no longer U1.11
- net RX-ARDUINO1: now also J15.2, U12.12; no longer J13.2, U9.11
- net RX-ARDUINO2: now also J26.2, U18.12; no longer J22.2, U14.11
- net RX-ARDUINO3: now also J37.2, U24.12; no longer J31.2, U19.11
- net RX-CELL: now also U1.4, U6.12; no longer U1.5, U5.12
- net RX-CELL1: now also U12.4, U7.12; no longer U6.12, U9.5
- net RX-CELL2: now also U13.12, U18.4; no longer U11.12, U14.5
- net RX-CELL3: now also U19.12, U24.4; no longer U16.12, U19.5
- net SCL-CELL: now also U4.5, U6.27; no longer U1.2, U5.27
- net SCL-CELL1: now also U11.5, U7.27; no longer U6.27, U9.2
- net SCL-CELL2: now also U13.27, U17.5; no longer U11.27, U14.2
- net SCL-CELL3: now also U19.27, U23.5; no longer U16.27, U19.2
- net SCL-QWIIC: now also J10.2, U4.8; no longer U1.13
- net SCL-QWIIC1: now also J13.4, J21.2, U11.8; no longer J11.4, U9.13
- net SCL-QWIIC2: now also J24.4, J32.2, U17.8; no longer J20.4, U14.13
- net SCL-QWIIC3: now also J35.4, J43.2, U23.8; no longer J29.4, U19.13
- net SDA-CELL: now also U4.4, U6.26; no longer U1.3, U5.26
- net SDA-CELL1: now also U11.4, U7.26; no longer U6.26, U9.3
- net SDA-CELL2: now also U13.26, U17.4; no longer U11.26, U14.3
- net SDA-CELL3: now also U19.26, U23.4; no longer U16.26, U19.3
- net SDA-QWIIC: now also J10.1, U4.1; no longer U1.12
- net SDA-QWIIC1: now also J13.3, J21.1, U11.1; no longer J11.3, U9.12
- net SDA-QWIIC2: now also J24.3, J32.1, U17.1; no longer J20.3, U14.12
- net SDA-QWIIC3: now also J35.3, J43.1, U23.1; no longer J29.3, U19.12
- net SHIELD1: now also J12.SHIELD, J12.SHIELD10, J12.SHIELD2, J12.SHIELD3, J12.SHIELD4, J12.SHIELD5, J12.SHIELD6, J12.SHIELD7, J12.SHIELD8, J12.SHIELD9; no longer J10.SHIELD, J10.SHIELD10, J10.SHIELD2, J10.SHIELD3, J10.SHIELD4, J10.SHIELD5, J10.SHIELD6, J10.SHIELD7, J10.SHIELD8, J10.SHIELD9
- net SHIELD2: now also J23.SHIELD, J23.SHIELD10, J23.SHIELD2, J23.SHIELD3, J23.SHIELD4, J23.SHIELD5, J23.SHIELD6, J23.SHIELD7, J23.SHIELD8, J23.SHIELD9; no longer J19.SHIELD, J19.SHIELD10, J19.SHIELD2, J19.SHIELD3, J19.SHIELD4, J19.SHIELD5, J19.SHIELD6, J19.SHIELD7, J19.SHIELD8, J19.SHIELD9
- net SHIELD3: now also J34.SHIELD, J34.SHIELD10, J34.SHIELD2, J34.SHIELD3, J34.SHIELD4, J34.SHIELD5, J34.SHIELD6, J34.SHIELD7, J34.SHIELD8, J34.SHIELD9; no longer J28.SHIELD, J28.SHIELD10, J28.SHIELD2, J28.SHIELD3, J28.SHIELD4, J28.SHIELD5, J28.SHIELD6, J28.SHIELD7, J28.SHIELD8, J28.SHIELD9
- net SIM_CLK: now also D6.6, J9.C3, U6.38; no longer D7.6, J8.C3, U5.38
- net SIM_CLK1: now also J16.C3, U7.38; no longer J14.C3, U6.38
- net SIM_CLK2: now also J27.C3, U13.38; no longer J23.C3, U11.38
- net SIM_CLK3: now also J38.C3, U19.38; no longer J32.C3, U16.38
- net SIM_IO: now also C17.1, D6.4, J9.C7, U6.39; no longer C16.1, D7.4, J8.C7, U5.39
- net SIM_IO1: now also J16.C7, U7.39; no longer J14.C7, U6.39
- net SIM_IO2: now also J27.C7, U13.39; no longer J23.C7, U11.39
- net SIM_IO3: now also J38.C7, U19.39; no longer J32.C7, U16.39
- net SIM_RST: now also C20.1, D6.3, J9.C2, U6.40; no longer C19.1, D7.3, J8.C2, U5.40
- net SIM_RST1: now also J16.C2, U7.40; no longer J14.C2, U6.40
- net SIM_RST2: now also J27.C2, U13.40; no longer J23.C2, U11.40
- net SIM_RST3: now also J38.C2, U19.40; no longer J32.C2, U16.40
- net TX-ARDUINO: now also U1.11; no longer U1.10
- net TX-ARDUINO1: now also J15.3, U12.11; no longer J13.3, U9.10
- net TX-ARDUINO2: now also J26.3, U18.11; no longer J22.3, U14.10
- net TX-ARDUINO3: now also J37.3, U24.11; no longer J31.3, U19.10
- net TX-CELL: now also U1.3, U6.13; no longer U1.4, U5.13
- net TX-CELL1: now also U12.3, U7.13; no longer U6.13, U9.4
- net TX-CELL2: now also U13.13, U18.3; no longer U11.13, U14.4
- net TX-CELL3: now also U19.13, U24.3; no longer U16.13, U19.4
- net VIN: now also D3.C, U5.5, U5.8; no longer D2.C, U4.5, U4.8
- net VIN1: now also D7.C, U9.5, U9.8; no longer D6.C, U8.5, U8.8
- net VIN2: now also U15.5, U15.8; no longer U13.5, U13.8
- net VIN3: now also U21.5, U21.8; no longer U18.5, U18.8
- net VSIM: now also D6.1, J9.C1, U6.41; no longer D7.1, J8.C1, U5.41
- net VSIM1: now also J16.C1, U7.41; no longer J14.C1, U6.41
- net VSIM2: now also J27.C1, U13.41; no longer J23.C1, U11.41
- net VSIM3: now also J38.C1, U19.41; no longer J32.C1, U16.41
- net VUSB_DET: now also JP6.2, U6.17; no longer JP7.2, U5.17
- net VUSB_DET1: now also JP9.2, U7.17; no longer JP1.2, U6.17
- net VUSB_DET2: now also U13.17; no longer U11.17
- net VUSB_DET3: now also U19.17; no longer U16.17
- net V_BATT: now also J11.2
- net V_BATT1: now also J14.2, J22.2, U8.3; no longer J12.2, U7.3
- net V_BATT2: now also J25.2, J33.2, U14.3; no longer J21.2, U12.3
- net V_BATT3: now also J36.2, J44.2, U20.3; no longer J30.2, U17.3
- net V_USB: now also D1.5, D3.A, JP6.1, R4.2; no longer D1.A, D5.5, JP7.1, R5.2
- net V_USB1: now also D7.A, J12.VBUS, JP9.1, R9.2, U8.4; no longer D6.A, J10.VBUS, JP1.1, R4.2, U7.4
- net V_USB2: now also J23.VBUS, U14.4; no longer J19.VBUS, U12.4
- net V_USB3: now also J34.VBUS, U20.4; no longer J28.VBUS, U17.4
Routing:
- net GPIO3-QWIIC2: track 0.00 -> 34.3 mm, vias 0 -> 1
- net GPIO3-QWIIC: track 0.00 -> 34.3 mm, vias 0 -> 1
- net GPIO3-QWIIC3: track 0.00 -> 34.3 mm, vias 0 -> 1
- net GPIO3-QWIIC1: track 0.00 -> 34.3 mm, vias 0 -> 1
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Other:
- board size 164.3 x 120.9 mm -> 162.8 x 120.9 mm
- board text added: "v11"
- board text removed: "x01"
